File: ovrBeaconGateway-btle.sch (KiCad schematic (older format))
At the start: 27 parts, among them J1 CONN_RJ45_RA, J2 CONN_1.27MM_5X2, Q1 FET_N_1.2A_20V, Q2 FET_N_1.2A_20V, U1 SILICONLABS_SI7050, U2 TOREX_XC6210, U3 LITEON_LTR-329ALS, U4 INTERSIL_ISL32602EFBZ, U5 BLUEGIGA_BLE121

Commit message: Added pricing and BOM
Parts:
- C5: footprint (none) -> ovrEngineered:C_0603
Changed lines of the file:
@@
 	7650 1500 8000 1500
 $Comp
-L +5V #PWR20
+L +5V #PWR01
 U 1 1 58B3312A
 P 7950 1250
-F 0 "#PWR20" H 7950 1100 50  0001 C CNN
+F 0 "#PWR01" H 7950 1100 50  0001 C CNN
 F 1 "+5V" H 7950 1390 50  0000 C CNN
 F 2 "" H 7950 1250 50  0000 C CNN
@@
 	7950 1300 7950 1250
 $Comp
-L GND #PWR21
+L GND #PWR02
 U 1 1 58B331C4
 P 7950 2000
-F 0 "#PWR21" H 7950 1750 50  0001 C CNN
+F 0 "#PWR02" H 7950 1750 50  0001 C CNN
 F 1 "GND" H 7950 1850 50  0000 C CNN
 F 2 "" H 7950 2000 50  0000 C CNN
@@
 Connection ~ 7950 1950
 $Comp
-L +3V3 #PWR18
+L +3V3 #PWR03
 U 1 1 58B3321D
 P 7350 1450
-F 0 "#PWR18" H 7350 1300 50  0001 C CNN
+F 0 "#PWR03" H 7350 1300 50  0001 C CNN
 F 1 "+3V3" H 7350 1590 50  0000 C CNN
 F 2 "" H 7350 1450 50  0000 C CNN
@@
 	7350 1500 7350 1450
 $Comp
-L GND #PWR16
+L GND #PWR04
 U 1 1 58B33268
 P 6700 2000
-F 0 "#PWR16" H 6700 1750 50  0001 C CNN
+F 0 "#PWR04" H 6700 1750 50  0001 C CNN
 F 1 "GND" H 6700 1850 50  0000 C CNN
 F 2 "" H 6700 2000 50  0000 C CNN
@@
 $EndComp
 $Comp
-L GND #PWR14
+L GND #PWR05
 U 1 1 58B33644
 P 6200 2250
-F 0 "#PWR14" H 6200 2000 50  0001 C CNN
+F 0 "#PWR05" H 6200 2000 50  0001 C CNN
 F 1 "GND" H 6200 2100 50  0000 C CNN
 F 2 "" H 6200 2250 50  0000 C CNN
@@
 $EndComp
 $Comp
-L +3V3 #PWR13
+L +3V3 #PWR06
 U 1 1 58B336C1
 P 6200 1150
-F 0 "#PWR13" H 6200 1000 50  0001 C CNN
+F 0 "#PWR06" H 6200 1000 50  0001 C CNN
 F 1 "+3V3" H 6200 1290 50  0000 C CNN
 F 2 "" H 6200 1150 50  0000 C CNN
@@
 $EndComp
 $Comp
-L +5V #PWR2
+L +5V #PWR07
 U 1 1 58B33CEE
 P 1600 1400
-F 0 "#PWR2" H 1600 1250 50  0001 C CNN
+F 0 "#PWR07" H 1600 1250 50  0001 C CNN
 F 1 "+5V" H 1600 1540 50  0000 C CNN
 F 2 "" H 1600 1400 50  0000 C CNN
@@
 $EndComp
 $Comp
-L GND #PWR3
+L GND #PWR08
 U 1 1 58B33D6E
 P 1600 1900
-F 0 "#PWR3" H 1600 1650 50  0001 C CNN
+F 0 "#PWR08" H 1600 1650 50  0001 C CNN
 F 1 "GND" H 1600 1750 50  0000 C CNN
 F 2 "" H 1600 1900 50  0000 C CNN
@@
 $EndComp
 $Comp
-L GND #PWR9
+L GND #PWR09
 U 1 1 58B33D94
 P 2650 1900
-F 0 "#PWR9" H 2650 1650 50  0001 C CNN
+F 0 "#PWR09" H 2650 1650 50  0001 C CNN
 F 1 "GND" H 2650 1750 50  0000 C CNN
 F 2 "" H 2650 1900 50  0000 C CNN
@@
 	1600 1800 1600 1900
 $Comp
-L +3V3 #PWR8
+L +3V3 #PWR010
 U 1 1 58B34078
 P 2650 1400
-F 0 "#PWR8" H 2650 1250 50  0001 C CNN
+F 0 "#PWR010" H 2650 1250 50  0001 C CNN
 F 1 "+3V3" H 2650 1540 50  0000 C CNN
 F 2 "" H 2650 1400 50  0000 C CNN
@@
 $EndComp
 $Comp
-L +3V3 #PWR4
+L +3V3 #PWR011
 U 1 1 58B347D6
 P 1650 3400
-F 0 "#PWR4" H 1650 3250 50  0001 C CNN
+F 0 "#PWR011" H 1650 3250 50  0001 C CNN
 F 1 "+3V3" H 1650 3540 50  0000 C CNN
 F 2 "" H 1650 3400 50  0000 C CNN
@@
 $EndComp
 $Comp
-L +3V3 #PWR19
+L +3V3 #PWR012
 U 1 1 58B34E3A
 P 7600 3750
-F 0 "#PWR19" H 7600 3600 50  0001 C CNN
+F 0 "#PWR012" H 7600 3600 50  0001 C CNN
 F 1 "+3V3" H 7600 3890 50  0000 C CNN
 F 2 "" H 7600 3750 50  0000 C CNN
@@
 $EndComp
 $Comp
-L GND #PWR17
+L GND #PWR013
 U 1 1 58B34E81
 P 6800 5000
-F 0 "#PWR17" H 6800 4750 50  0001 C CNN
+F 0 "#PWR013" H 6800 4750 50  0001 C CNN
 F 1 "GND" H 6800 4850 50  0000 C CNN
 F 2 "" H 6800 5000 50  0000 C CNN
@@
 $EndComp
 $Comp
-L +3V3 #PWR15
+L +3V3 #PWR014
 U 1 1 58B350CF
 P 6400 3400
-F 0 "#PWR15" H 6400 3250 50  0001 C CNN
+F 0 "#PWR014" H 6400 3250 50  0001 C CNN
 F 1 "+3V3" H 6400 3540 50  0000 C CNN
 F 2 "" H 6400 3400 50  0000 C CNN
@@
 $EndComp
 $Comp
-L GND #PWR1
+L GND #PWR015
 U 1 1 58B364F1
 P 1350 6850
-F 0 "#PWR1" H 1350 6600 50  0001 C CNN
+F 0 "#PWR015" H 1350 6600 50  0001 C CNN
 F 1 "GND" H 1350 6700 50  0000 C CNN
 F 2 "" H 1350 6850 50  0000 C CNN
@@
 $EndComp
 $Comp
-L +3V3 #PWR5
+L +3V3 #PWR016
 U 1 1 58B3654C
 P 2050 6600
-F 0 "#PWR5" H 2050 6450 50  0001 C CNN
+F 0 "#PWR016" H 2050 6450 50  0001 C CNN
 F 1 "+3V3" H 2050 6740 50  0000 C CNN
 F 2 "" H 2050 6600 50  0000 C CNN
@@
 $EndComp
 $Comp
-L +3V3 #PWR10
+L +3V3 #PWR017
 U 1 1 58B36B31
 P 3150 6500
-F 0 "#PWR10" H 3150 6350 50  0001 C CNN
+F 0 "#PWR017" H 3150 6350 50  0001 C CNN
 F 1 "+3V3" H 3150 6640 50  0000 C CNN
 F 2 "" H 3150 6500 50  0000 C CNN
@@
 Connection ~ 1650 3550
 $Comp
-L GND #PWR6
+L GND #PWR018
 U 1 1 58B37DC3
 P 2450 4600
-F 0 "#PWR6" H 2450 4350 50  0001 C CNN
+F 0 "#PWR018" H 2450 4350 50  0001 C CNN
 F 1 "GND" H 2450 4450 50  0000 C CNN
 F 2 "" H 2450 4600 50  0000 C CNN
@@
 SCL
 $Comp
-L GND #PWR22
+L GND #PWR019
 U 1 1 58B39AD3
 P 8150 3850
-F 0 "#PWR22" H 8150 3600 50  0001 C CNN
+F 0 "#PWR019" H 8150 3600 50  0001 C CNN
 F 1 "GND" H 8150 3700 50  0000 C CNN
 F 2 "" H 8150 3850 50  0000 C CNN
@@
 $EndComp
 $Comp
-L +3V3 #PWR12
+L +3V3 #PWR020
 U 1 1 58B3A862
 P 5750 6450
-F 0 "#PWR12" H 5750 6300 50  0001 C CNN
+F 0 "#PWR020" H 5750 6300 50  0001 C CNN
 F 1 "+3V3" H 5750 6590 50  0000 C CNN
 F 2 "" H 5750 6450 50  0000 C CNN
@@
 $EndComp
 $Comp
-L GND #PWR11
+L GND #PWR021
 U 1 1 58B3A8B8
 P 5050 6700
-F 0 "#PWR11" H 5050 6450 50  0001 C CNN
+F 0 "#PWR021" H 5050 6450 50  0001 C CNN
 F 1 "GND" H 5050 6550 50  0000 C CNN
 F 2 "" H 5050 6700 50  0000 C CNN
@@
 $EndComp
 $Comp
-L +3V3 #PWR24
+L +3V3 #PWR022
 U 1 1 58B3F6FC
 P 9950 3950
-F 0 "#PWR24" H 9950 3800 50  0001 C CNN
+F 0 "#PWR022" H 9950 3800 50  0001 C CNN
 F 1 "+3V3" H 9950 4090 50  0000 C CNN
 F 2 "" H 9950 3950 50  0000 C CNN
@@
 $EndComp
 $Comp
-L GND #PWR23
+L GND #PWR023
 U 1 1 58B3F873
 P 9200 4250
-F 0 "#PWR23" H 9200 4000 50  0001 C CNN
+F 0 "#PWR023" H 9200 4000 50  0001 C CNN
 F 1 "GND" H 9200 4100 50  0000 C CNN
 F 2 "" H 9200 4250 50  0000 C CNN
@@
 F 0 "C5" H 2250 6650 60  0000 C CNN
 F 1 "C_0.1uF_10v_0603" H 2250 6550 60  0001 C CNN
-F 2 "" H 2500 6650 60  0001 C CNN
+F 2 "ovrEngineered:C_0603" H 2500 6650 60  0001 C CNN
 F 3 "http://search.murata.co.jp/Ceramy/image/img/A01X/G101/ENG/GRM188R71C104KA01-01.pdf" H 2450 6350 60  0001 C CNN
 F 4 "Murata" H 1950 6450 60  0001 C CNN "Manufacturer"
@@
 $EndComp
 $Comp
-L GND #PWR7
+L GND #PWR024
 U 1 1 58B440C1
 P 2450 6700
-F 0 "#PWR7" H 2450 6450 50  0001 C CNN
+F 0 "#PWR024" H 2450 6450 50  0001 C CNN
 F 1 "GND" H 2450 6550 50  0000 C CNN
 F 2 "" H 2450 6700 50  0000 C CNN

Commit message: Out for DFM
Parts:
- removed C3: C_10000pF_25v_0603, ovrEngineered:C_0603, symbol C_10000pF_25v_0603
- removed D3: LED_RED_0603, ovrEngineered:D_0603, symbol LED_RED_0603
- removed Q2: FET_N_1.2A_20V, ovrEngineered:FET_N_1.2A_20V, symbol FET_N_1.2A_20V
- removed R3: R_402_1%_0603, ovrEngineered:R_0603, symbol R_402_1%_0603
- removed R6, R7, R8, R9: R_10K_1%_0603, ovrEngineered:R_0603, symbol R_10K_1%_0603
- added U6: MIC803-29D4VM3, ovrEngineered:SOT-23-3, symbol MIC803-29D4VM3
Connections:
- net +3V3: now also U4.4 (DE), U6.3 (VCC)
- net GND: now also U4.3 (~RE), U6.1 (GND); no longer U5.15 (GND)
- net ~RESET: now also U6.2 (~RESET)
- net 422_DE: no longer names the net of U5.6 (P0_0)
- net 422_DE: no longer U4.4 (DE)
- net LED_ERROR: no longer names the net of U5.12 (P0_7)
- net ~422_RE: no longer names the net of U5.5 (P0_1)
- net ~422_RE: no longer U4.3 (~RE)
- no-connect marks 10 -> 15
